File: FPGA-main-d.sch (KiCad schematic (older format))
At the start: 25 parts, among them U1 XC7A75T-FTG256

Commit message: Add wire up for Q-SPI flash module.
Connections:
- net +1V8 is gone; now on net GND: U1.F8 (VCCBATT_0)
Changed lines of the file:
@@
 Connection ~ 11650 4725
-$Comp
-L power:+1V8 #PWR0169
-U 1 1 60F30312
-P 7375 5425
-F 0 "#PWR0169" H 7375 5275 50  0001 C CNN
-F 1 "+1V8" V 7390 5553 50  0000 L CNN
-F 2 "" H 7375 5425 50  0001 C CNN
-F 3 "" H 7375 5425 50  0001 C CNN
-	1    7375 5425
-	0    -1   -1   0
-$EndComp
 $Comp
 L Device:C_Small C?
@@
 Text GLabel 5575 5525 1    50   Input ~ 0
 VCCBRAM
+$Comp
+L power:GND #PWR0184
+U 1 1 60C049C3
+P 7375 5425
+F 0 "#PWR0184" H 7375 5175 50  0001 C CNN
+F 1 "GND" V 7380 5297 50  0000 R CNN
+F 2 "" H 7375 5425 50  0001 C CNN
+F 3 "" H 7375 5425 50  0001 C CNN
+	1    7375 5425
+	0    1    1    0
+$EndComp
 $EndSCHEMATC
